File: ZK3-BP-MOD.kicad_sch (KiCad schematic)
At the start: 32 parts, among them J28 R, J32 R, J33 R, J35 R, J36 R, U1 YAAJ_BluePill_Part_Like_SWD_B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

Commit message: Fix C3 C4
Parts:
- renumbered C4 to C3, C3 to C4
